File: hardware/LEC011102.kicad_sch (KiCad schematic)
At the start: 40 parts, among them J1 Button, J2 PWR, J3 CONTACT_1, J4 CONTACT_2, K1 HK19F-5V, Q1 S8050, U1 MC78M05_TO252, U2 NE555D

Commit message: Add prod files
Parts:
- C1, C7: JLCPCB_CORRECTION 0;0;180 -> 0;0;0
- C3: JLCPCB_CORRECTION (none) -> 0;0;0
- D1: JLCPCB_CORRECTION 0;0;90 -> 0;0;0
- J1: JLCPCB_CORRECTION (none) -> 2.54;0;180
- J2: JLCPCB_CORRECTION (none) -> 2.54;0;0
- J3, J4: JLCPCB_CORRECTION (none) -> 0;0;180
- RV1: JLCPCB_CORRECTION 0;0;180 -> -2.54;0;180
Changed lines of the file:
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@@
+      (effects (font (size 1.27 1.27)) hide)
+    )
+    (property "JLCPCB_CORRECTION" "0;0;0" (id 8) (at 86.36 132.08 0)
       (effects (font (size 1.27 1.27)) hide)
     )
@@
       (effects (font (size 1.27 1.27)) hide)
     )
-    (property "JLCPCB_CORRECTION" "0;0;90" (id 6) (at 52.07 30.48 0)
+    (property "JLCPCB_CORRECTION" "0;0;0" (id 6) (at 52.07 30.48 0)
       (effects (font (size 1.27 1.27)) hide)
     )
@@
       (effects (font (size 1.27 1.27)) hide)
     )
-    (property "JLCPCB_CORRECTION" "0;0;180" (id 6) (at 69.85 34.29 0)
+    (property "JLCPCB_CORRECTION" "0;0;0" (id 6) (at 69.85 34.29 0)
       (effects (font (size 1.27 1.27)) hide)
     )
@@
       (effects (font (size 1.27 1.27)) hide)
     )
-    (property "JLCPCB_CORRECTION" "0;0;180" (id 6) (at 127 34.29 0)
+    (property "JLCPCB_CORRECTION" "0;0;0" (id 6) (at 127 34.29 0)
       (effects (font (size 1.27 1.27)) hide)
     )
@@
       (effects (font (size 1.27 1.27)) hide)
     )
+    (property "JLCPCB_CORRECTION" "2.54;0;0" (id 8) (at 35.56 31.75 0)
+      (effects (font (size 1.27 1.27)) hide)
+    )
     (pin "1")
     (pin "2")
@@
       (effects (font (size 1.27 1.27)) hide)
     )
-    (property "JLCPCB_CORRECTION" "0;0;180" (id 7) (at 86.36 92.71 0)
+    (property "JLCPCB_CORRECTION" "-2.54;0;180" (id 7) (at 86.36 92.71 0)
       (effects (font (size 1.27 1.27)) hide)
     )
@@
       (effects (font (size 1.27 1.27)) hide)
     )
+    (property "JLCPCB_CORRECTION" "0;0;180" (id 9) (at 260.35 81.28 0)
+      (effects (font (size 1.27 1.27)) hide)
+    )
     (pin "1")
     (pin "2")
@@
     )
     (property "Comment" "Genuine only" (id 8) (at 260.35 92.71 0)
+      (effects (font (size 1.27 1.27)) hide)
+    )
+    (property "JLCPCB_CORRECTION" "0;0;180" (id 9) (at 260.35 92.71 0)
       (effects (font (size 1.27 1.27)) hide)
     )
@@
       (effects (font (size 1.27 1.27)) hide)
     )
+    (property "JLCPCB_CORRECTION" "2.54;0;180" (id 8) (at 22.86 118.11 0)
+      (effects (font (size 1.27 1.27)) hide)
+    )
